File: Hardware /Cendit11713-v2/MainBoard.Pic18F4550.Option2/MainBoard .Backup.kicad_pcb (KiCad board)
At the start: 2 copper layers, 86 parts, among them CON1 POWER_BUS, CON2 ICSP_CON, CON3 USB_CON, J1 RESET_CON, J2 SATA_PLUG _22P_SMT, J4 SATA_PLUG _22P_SMT, P1 DEBUG_HEADER_21P, P2 DEBUG_HEADER_21P, Q1 2N2222, U1 PIC18F4550-I/P, U3 PCF85263A, Y1 Crystal, Y2 32.768KHZ

Commit message: Respaldo rapido
Parts:
- moved J4 3.94 mm to (153.2, 75.4)
- moved P1 2.44 mm to (161.9, 67.4)
Connections:
- CON1 pad 1: /VDD_3V -> /VPWR
- CON1 pad 10: Net-(CON1-Pad10) -> GNDD
- CON1 pad 2: GNDD -> GNDPWR
- CON1 pad 3: GNDD -> /VCC_5V
- CON1 pad 5: /VCC_5V -> /VDD_3V
- CON1 pad 6: Net-(CON1-Pad6) -> GNDD
- CON1 pad 7: GNDPWR -> Net-(CON1-Pad7)
- CON1 pad 9: /VPWR -> Net-(CON1-Pad9)
- J2 pad 1: /VPWR -> //RST_KEY
- J2 pad 10: //RST_LAN -> /PB0
- J2 pad 11: //RST_VIKING -> /PB1
- J2 pad 12: //CS_LAN -> /PB2
- J2 pad 13: //CS_VIKING -> /PB3
- J2 pad 14: GNDD -> /PB4
- J2 pad 15: /PB0 -> /PB6
- J2 pad 16: /PB1 -> /PB7
- J2 pad 17: /PB2 -> /VCC_3V
- J2 pad 18: /PB3 -> GNDD
- J2 pad 19: /PB4 -> /VCC_5V
- J2 pad 2: /GND_PWR -> //RST_GPIB
- J2 pad 20: /PB6 -> /GND_PWR
- J2 pad 21: /PB7 -> /VPWR
- J2 pad 3: /VCC_5V -> /MISO
- J2 pad 4: GNDD -> /MOSI
- J2 pad 5: /VCC_3V -> //RST_LAN
- J2 pad 6: //RST_KEY -> //RST_VIKING
- J2 pad 7: //RST_GPIB -> //CS_LAN
- J2 pad 8: /MISO -> //CS_VIKING
- J2 pad 9: /MOSI -> GNDD
- J4 pad 1: /PA0 -> Net-(J4-Pad1)
- J4 pad 10: GNDD -> /PA3
- J4 pad 11: /PC0 -> /PA4
- J4 pad 12: /PC1 -> /PA5
- J4 pad 13: /PC2 -> /PE0
- J4 pad 14: /PD0 -> /PE1
- J4 pad 15: /PD1 -> /PE2
- J4 pad 17: /VDD_3V -> /PC0
- J4 pad 18: GNDD -> /PC1
- J4 pad 19: /VCC_5V -> /PC2
- J4 pad 2: /PA1 -> /VPWR
- J4 pad 20: GNDPWR -> /PD0
- J4 pad 21: /VPWR -> /PD1
- J4 pad 3: /PA2 -> GNDPWR
- J4 pad 4: /PA3 -> /VCC_5V
- J4 pad 5: /PA4 -> GNDD
- J4 pad 6: /PA5 -> /VDD_3V
- J4 pad 7: /PE0 -> /PA0
- J4 pad 8: /PE1 -> /PA1
- J4 pad 9: /PE2 -> /PA2
- P1 pad 1: /PA0 -> /VPWR
- P1 pad 10: GNDD -> /PA4
- P1 pad 11: /PC0 -> /PA5
- P1 pad 12: /PC1 -> /PE0
- P1 pad 13: /PC2 -> /PE1
- P1 pad 14: /PD0 -> /PE2
- P1 pad 15: /PD1 -> GNDD
- P1 pad 16: GNDD -> /PC0
- P1 pad 17: /VDD_3V -> /PC1
- P1 pad 18: GNDD -> /PC2
- P1 pad 19: /VCC_5V -> /PD0
- P1 pad 2: /PA1 -> GNDPWR
- P1 pad 20: GNDPWR -> /PD1
- P1 pad 21: /VPWR -> /GND
- P1 pad 3: /PA2 -> /VCC_5V
- P1 pad 4: /PA3 -> GNDD
- P1 pad 5: /PA4 -> /VDD_3V
- P1 pad 6: /PA5 -> /PA0
- P1 pad 7: /PE0 -> /PA1
- P1 pad 8: /PE1 -> /PA2
- P1 pad 9: /PE2 -> /PA3
- P2 pad 1: /PB7 -> /VPWR
- P2 pad 10: //CS_LAN -> /PB2
- P2 pad 11: //RST_VIKING -> /PB1
- P2 pad 12: //RST_LAN -> /PB0
- P2 pad 13: /MOSI -> GNDD
- P2 pad 14: /MISO -> //CS_VIKING
- P2 pad 15: //RST_GPIB -> //CS_LAN
- P2 pad 16: //RST_KEY -> //RST_VIKING
- P2 pad 17: /VDD_3V -> //RST_LAN
- P2 pad 18: GNDD -> /MOSI
- P2 pad 19: /VCC_5V -> /MISO
- P2 pad 2: /PB6 -> /GND_PWR
- P2 pad 20: /GND_PWR -> //RST_GPIB
- P2 pad 21: /VPWR -> //RST_KEY
- P2 pad 3: /PB4 -> /VCC_5V
- P2 pad 4: /PB3 -> GNDD
- P2 pad 5: /PB2 -> /VDD_3V
- P2 pad 6: /PB1 -> /PB7
- P2 pad 7: /PB0 -> /PB6
- P2 pad 8: GNDD -> /PB4
- P2 pad 9: //CS_VIKING -> /PB3
Routing:
- net GNDD: track 180.6 -> 305.3 mm, vias 6 -> 9
- net /VCC_5V: track 21.6 -> 139.7 mm, vias 0 -> 3
- net /VPWR: track 9.55 -> 111.0 mm, vias 1 -> 2
- net /VDD_3V: track 19.7 -> 96.5 mm, vias 0 -> 3
- net GNDPWR: track 40.5 -> 115.2 mm
- net /GND_PWR: track 0.00 -> 14.3 mm
- net /PD1: track 41.6 -> 30.2 mm
- net /PB1: track 31.2 -> 42.3 mm
- net /PD0: track 39.7 -> 28.9 mm
- net /PC0: track 35.9 -> 25.1 mm
- net /PC1: track 36.5 -> 26.9 mm
- net /PC2: track 36.8 -> 27.6 mm
- net /PB0: track 30.8 -> 39.9 mm
- net /PB2: track 30.1 -> 39.0 mm
- net //CS_VIKING: track 32.1 -> 39.2 mm
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- added copper zone on F.Cu, net GNDD
