File: Hardware /Cendit11713-v2/ArchivosGerber/VikingPortExpandeMC33996/KicadFiles/PortExpanderMC33996.sch (KiCad schematic (older format))
At the start: 12 parts, among them J1 DEBUG_CONN, P1 VIKING_HEADER_9P, P2 VIKING_HEADER_9P, U1 MC33996EKR2

Commit message: Trabajo en CenditLab + Cendit11713
  - Diseño + codigo UI
  - PCBs tarjeta madre + puertos Viking
  - Se generan Gerber para solicitud de prototipos PCB
Parts:
- removed R1: RL, Resistors_SMD:R_0805_HandSoldering, symbol R_Small
- C1, C3: footprint Capacitors_SMD:c_elec_3x5.3 -> Capacitors_SMD:C_1206_HandSoldering
Connections:
- wire segments 93 -> 92
Changed lines of the file:
@@
 EELAYER 25 0
 EELAYER END
-$Descr A4 11693 8268
+$Descr USLetter 11000 8500
 encoding utf-8
 Sheet 1 1
-Title ""
-Date ""
-Rev ""
-Comp ""
-Comment1 ""
-Comment2 ""
-Comment3 ""
+Title "Expansor de puertos Viking"
+Date "2017-11-23"
+Rev "Rev 1"
+Comp "CENDIT"
+Comment1 "Jose Arias"
+Comment2 "Proyecto TEG"
+Comment3 "UCV"
 Comment4 ""
 $EndDescr
@@
 F 0 "C1" H 1575 5050 50  0000 L CNN
 F 1 "10uF" H 1575 4850 50  0000 L CNN
-F 2 "Capacitors_SMD:c_elec_3x5.3" H 1588 4800 50  0001 C CNN
+F 2 "Capacitors_SMD:C_1206_HandSoldering" H 1588 4800 50  0001 C CNN
 F 3 "" H 1550 4950 50  0001 C CNN
 	1    1550 4950
@@
 $EndComp
 Wire Bus Line
-	2450 1750 2450 3100
+	2450 1100 2450 3100
 Wire Wire Line
 	2000 2100 1900 2100
@@
 F 0 "C3" H 2425 5050 50  0000 L CNN
 F 1 "10uF" H 2425 4850 50  0000 L CNN
-F 2 "Capacitors_SMD:c_elec_3x5.3" H 2438 4800 50  0001 C CNN
+F 2 "Capacitors_SMD:C_1206_HandSoldering" H 2438 4800 50  0001 C CNN
 F 3 "" H 2400 4950 50  0001 C CNN
 	1    2400 4950
@@
 Wire Wire Line
 	1950 3550 1650 3550
-$Comp
-L R_Small R1
-U 1 1 59DED0AD
-P 4500 3600
-F 0 "R1" H 4530 3620 50  0000 L CNN
-F 1 "RL" H 4530 3560 50  0000 L CNN
-F 2 "Resistors_SMD:R_0805_HandSoldering" H 4500 3600 50  0001 C CNN
-F 3 "" H 4500 3600 50  0000 C CNN
-	1    4500 3600
-	1    0    0    -1
-$EndComp
-Wire Wire Line
-	4500 3350 4500 3500
-Wire Wire Line
-	4500 3700 4500 3950
+Wire Wire Line
+	4500 3350 4500 3950
 $Comp
 L CONN_01X09 P1
@@
 Wire Wire Line
 	5000 2150 4900 2150
-Text Label 4500 3800 0    60   ~ 0
+Text Label 2600 3950 0    60   ~ 0
 MISO
 Entry Wire Line
@@
 Text Label 4350 3150 0    60   ~ 0
 P15
-Text Label 4800 1450 0    60   ~ 0
+Text Label 4800 2050 0    60   ~ 0
 P0
-Text Label 4800 1550 0    60   ~ 0
+Text Label 4800 1950 0    60   ~ 0
 P1
-Text Label 4800 1650 0    60   ~ 0
+Text Label 4800 1850 0    60   ~ 0
 P2
 Text Label 4800 1750 0    60   ~ 0
 P3
-Text Label 4800 1850 0    60   ~ 0
+Text Label 4800 1650 0    60   ~ 0
 P4
-Text Label 4800 1950 0    60   ~ 0
+Text Label 4800 1550 0    60   ~ 0
 P5
-Text Label 4800 2050 0    60   ~ 0
+Text Label 4800 1450 0    60   ~ 0
 P6
-Text Label 4800 2450 0    60   ~ 0
+Text Label 4800 3250 0    60   ~ 0
 P7
-Text Label 4800 2550 0    60   ~ 0
+Text Label 4800 3150 0    60   ~ 0
 P8
-Text Label 4800 2650 0    60   ~ 0
+Text Label 4800 3050 0    60   ~ 0
 P9
-Text Label 4800 2750 0    60   ~ 0
+Text Label 4800 2950 0    60   ~ 0
 P10
 Text Label 4800 2850 0    60   ~ 0
 P11
-Text Label 4800 2950 0    60   ~ 0
+Text Label 4800 2750 0    60   ~ 0
 P12
-Text Label 4800 3050 0    60   ~ 0
+Text Label 4800 2650 0    60   ~ 0
 P13
-Text Label 4800 3150 0    60   ~ 0
+Text Label 4800 2550 0    60   ~ 0
 P14
-Text Label 4800 3250 0    60   ~ 0
+Text Label 4800 2450 0    60   ~ 0
 P15
 Wire Wire Line
@@
 	-1   0    0    -1
 $EndComp
+Wire Bus Line
+	2450 1100 4650 1100
 $EndSCHEMATC
