File: Hardware /Cendit11713-v2/PortExpanderMC33996.Single.Option1/PortExpanderMC33996.sch (KiCad schematic (older format))
At the start: 12 parts, among them J1 DEBUG_CONN, P1 VIKING_HEADER_9P, P2 VIKING_HEADER_9P, U1 MC33996EKR2

Commit message: En Cendit11713 + CenditLab respaldo
  - Se revisan tarjetas
  - Correccion en PCB GPIB
  - Se inicia tarjeta madre en una pieza (MainBoard.OnePiece)
Parts:
- C1, C3: footprint Capacitors_SMD:c_elec_3x5.3 -> Capacitors_SMD:C_1210_HandSoldering
Changed lines of the file:
@@
 F 0 "C1" H 1575 5050 50  0000 L CNN
 F 1 "10uF" H 1575 4850 50  0000 L CNN
-F 2 "Capacitors_SMD:c_elec_3x5.3" H 1588 4800 50  0001 C CNN
+F 2 "Capacitors_SMD:C_1210_HandSoldering" H 1588 4800 50  0001 C CNN
 F 3 "" H 1550 4950 50  0001 C CNN
 	1    1550 4950
@@
 F 0 "C3" H 2425 5050 50  0000 L CNN
 F 1 "10uF" H 2425 4850 50  0000 L CNN
-F 2 "Capacitors_SMD:c_elec_3x5.3" H 2438 4800 50  0001 C CNN
+F 2 "Capacitors_SMD:C_1210_HandSoldering" H 2438 4800 50  0001 C CNN
 F 3 "" H 2400 4950 50  0001 C CNN
 	1    2400 4950
